File: Industrial-Protocol-Auditor-Hardware/Industrial-Protocol-Auditor-Hardware.kicad_pcb (KiCad board)
At the start: 2 copper layers, 111.5 x 60.4 mm, 94 parts, among them J1 Jack-DC, J2 USB_C_Receptacle, J3 RS_Port, J4 Batt_Port, J5 CAN_Port, J6 Conn_01x08, J7 E07-M1101D-SMA, M1 Motor_DC, Q1 AO3400A, SW1 UP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

Commit message: Finished the PCB design and created production files to get a price in JLCPCB webpage.
Parts:
- moved R31 2.25 mm to (144.5, 108.3), turned to 90 degrees
- moved R30 1.65 mm to (155.5, 108.3), turned to 90 degrees
- moved C9 1.60 mm to (155.4, 115.7), turned to 90 degrees
- moved C17 1.58 mm to (142.9, 109.9)
Routing:
- net +3V3: track 1.51 -> 259.9 mm, vias 0 -> 10
- net /RF_GDO2: track 0.00 -> 139.2 mm, vias 0 -> 1
- net Net-(R29-Pad2): track 0.00 -> 105.4 mm, vias 0 -> 2
- net /RF_GDO0: track 0.00 -> 105.3 mm, vias 0 -> 1
- net /TFT_DC: track 0.00 -> 92.5 mm, vias 0 -> 1
- net /~{DS_RST}: track 0.00 -> 89.4 mm, vias 0 -> 4
- net /SW_OK: track 0.00 -> 79.2 mm, vias 0 -> 5
- net /SW_UP: track 0.00 -> 71.1 mm, vias 0 -> 4
- net /SW_LEF: track 0.00 -> 70.0 mm, vias 0 -> 4
- net /CAN_Rx: track 0.00 -> 69.4 mm, vias 0 -> 2
- net /CLK: track 0.00 -> 66.7 mm, vias 0 -> 2
- net /MOSI: track 0.00 -> 64.9 mm, vias 0 -> 2
- net /VBAT: track 0.00 -> 64.2 mm
- net /SW_RIG: track 0.00 -> 63.8 mm, vias 0 -> 4
- net /SW_DWN: track 0.00 -> 61.5 mm, vias 0 -> 4
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